File: BMS-Cell-Module-Circuit/BMS_Cell_Module.kicad_pcb (KiCad board)
At the start: 2 copper layers, 45.7 x 65.8 mm, 35 parts, among them J1 Conn_01x02_Female, J2 Conn_01x04_Female, J3 Conn_01x04_Female, M1 SI2312BDS-T1-E3, U2 ADUM1250ARZ, U3 ATTINY85V-10SU 8S2 EIAJ SOIC

Commit message: Minor tweaks
Parts:
- R3: value 20K -> 68K
Changed lines of the file:
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@@
       (effects (font (size 1 1) (thickness 0.15)))
     )
-    (fp_text value 20K (at 0.1143 1.7907) (layer F.Fab)
+    (fp_text value 68K (at 0.1143 1.7907) (layer F.Fab)
       (effects (font (size 1 1) (thickness 0.15)))
     )

Commit message: Minor amends
Parts:
- R3: value 68K -> 20K
Other:
- board text added: "(c)2017 Stuart Pittaway #MadeInTheBlackCountry"
- board text added: "Version 2.1 (Mar 2018)"
- board text removed: "Version 2 (Dec 2017)"
Changed lines of the file:
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@@
   )
   (setup
-    (last_trace_width 0.35)
+    (last_trace_width 1)
     (user_trace_width 0.5)
     (user_trace_width 1)
     (trace_clearance 0.3)
-    (zone_clearance 0.508)
+    (zone_clearance 0.8)
     (zone_45_only no)
     (trace_min 0.35)
@@
     (add_net "Net-(R5-Pad2)")
   )
+  (module ATTINY:DO-221AC (layer F.Cu)
+    (at 133.985 114.3254 90)
+    (fp_text reference D1 (at -0.254 0 90) (layer F.SilkS) hide
+      (effects (font (size 1.25 1.25) (thickness 0.25)))
+    )
+    (fp_text value SE30AFG-M3/6A (at 0.381 -2.286 270) (layer F.Fab)
+      (effects (font (size 1 1) (thickness 0.25)))
+    )
+    (fp_line (start 2.2 -1.35) (end 2.2 -1.1) (layer F.SilkS) (width 0.2))
+    (fp_line (start 2.2 1.35) (end 2.2 1.1) (layer F.SilkS) (width 0.2))
+    (fp_line (start -2.2 1.35) (end -2.2 1.1) (layer F.SilkS) (width 0.2))
+    (fp_line (start -2.2 -1.35) (end -2.2 -1.1) (layer F.SilkS) (width 0.2))
+    (fp_line (start 1.286 -1.25) (end 1.286 1.25) (layer F.SilkS) (width 0.2))
+    (fp_line (start -2.175 -1.35) (end 2.175 -1.35) (layer F.SilkS) (width 0.2))
+    (fp_line (start -2.175 1.35) (end 2.175 1.35) (layer F.SilkS) (width 0.2))
+    (pad 1 smd rect (at 2.16 0 90) (size 1.2 1.52) (layers F.Cu F.Paste F.Mask)
+      (net 3 "Net-(D1-Pad1)"))
+    (pad 2 smd rect (at -2.16 0 90) (size 1.2 1.52) (layers F.Cu F.Paste F.Mask)
+      (net 6 BATT+RAW))
+    (model "/Library/Application Support/kicad/packages3d/Diodes_SMD.3dshapes/SMA_Standard.wrl"
+      (at (xyz 0 0 0))
+      (scale (xyz 0.35 0.35 0.25))
+      (rotate (xyz 0 0 0))
+    )
+  )
   (module Connectors:1pin (layer F.Cu)
     (at 174.2694 123.3932)
@@
       (effects (font (size 1 1) (thickness 0.15)))
     )
-    (fp_text value 68K (at 0.1143 1.7907) (layer F.Fab)
+    (fp_text value 20K (at 0.1143 1.7907) (layer F.Fab)
       (effects (font (size 1 1) (thickness 0.15)))
     )
@@
       (at (xyz 0 0 0))
       (scale (xyz 1 1 1))
-      (rotate (xyz 0 0 0))
-    )
-  )
-  (module ATTINY:DO-221AC (layer F.Cu)
-    (at 133.985 114.3254 90)
-    (fp_text reference D1 (at -4.5974 -1.1684 90) (layer F.SilkS)
-      (effects (font (size 1.5 1.5) (thickness 0.25)))
-    )
-    (fp_text value SE30AFG-M3/6A (at -0.1016 -10.1346 180) (layer F.Fab)
-      (effects (font (size 1 1) (thickness 0.25)))
-    )
-    (fp_line (start 2.2 -1.35) (end 2.2 -1.1) (layer F.SilkS) (width 0.2))
-    (fp_line (start 2.2 1.35) (end 2.2 1.1) (layer F.SilkS) (width 0.2))
-    (fp_line (start -2.2 1.35) (end -2.2 1.1) (layer F.SilkS) (width 0.2))
-    (fp_line (start -2.2 -1.35) (end -2.2 -1.1) (layer F.SilkS) (width 0.2))
-    (fp_line (start -1 -1.25) (end -1 1.25) (layer F.SilkS) (width 0.2))
-    (fp_line (start -2.175 -1.35) (end 2.175 -1.35) (layer F.SilkS) (width 0.2))
-    (fp_line (start -2.175 1.35) (end 2.175 1.35) (layer F.SilkS) (width 0.2))
-    (pad 1 smd rect (at 2.16 0 90) (size 1.2 1.52) (layers F.Cu F.Paste F.Mask)
-      (net 3 "Net-(D1-Pad1)"))
-    (pad 2 smd rect (at -2.16 0 90) (size 1.2 1.52) (layers F.Cu F.Paste F.Mask)
-      (net 6 BATT+RAW))
-    (model "/Library/Application Support/kicad/packages3d/Diodes_SMD.3dshapes/SMA_Standard.wrl"
-      (at (xyz 0 0 0))
-      (scale (xyz 0.35 0.35 0.25))
       (rotate (xyz 0 0 0))
     )
@@
     (effects (font (size 1.5 1.5) (thickness 0.3)) (justify mirror))
   )
-  (gr_text "(c)2017 Stuart Pittaway" (at 150.876 90.9828 90) (layer B.SilkS)
+  (gr_text "(c)2017 Stuart Pittaway\n\n#MadeInTheBlackCountry" (at 140.3096 94.7166 90) (layer B.SilkS)
     (effects (font (size 1.5 1.5) (thickness 0.3)) (justify mirror))
   )
@@
   (gr_line (start 131.2926 126.238) (end 177.038 126.238) (layer Edge.Cuts) (width 0.15))
   (gr_line (start 131.2926 60.452) (end 131.2926 126.238) (layer Edge.Cuts) (width 0.15))
-  (gr_text "Version 2 (Dec 2017)" (at 175.6918 110.5408 90) (layer F.SilkS)
+  (gr_text "Version 2.1 (Mar 2018)" (at 175.6918 110.5408 90) (layer F.SilkS)
     (effects (font (size 1 1) (thickness 0.25)))
   )
@@
     (effects (font (size 1.5 1.5) (thickness 0.3)))
   )
-  (gr_text DIYBMS (at 172.339 99.5172) (layer F.SilkS)
+  (gr_text DIYBMS (at 172.0342 99.949) (layer F.SilkS)
     (effects (font (size 1.5 1.5) (thickness 0.3)))
   )
@@
   (segment (start 160.4782 119.3028) (end 160.6804 119.1006) (width 0.35) (layer F.Cu) (net 6) (status 30))
   (segment (start 160.5788 103.7016) (end 160.1028 103.2256) (width 0.35) (layer F.Cu) (net 6) (status 30))
-  (segment (start 149.1996 80.6704) (end 136.2202 80.6704) (width 0.35) (layer B.Cu) (net 7))
+  (segment (start 149.1996 80.6704) (end 136.2202 80.6704) (width 1) (layer B.Cu) (net 7))
   (segment (start 135.922 80.3722) (end 133.9342 80.3722) (width 0.35) (layer F.Cu) (net 7))
   (segment (start 136.0932 80.5434) (end 135.922 80.3722) (width 0.35) (layer F.Cu) (net 7))
@@
   (segment (start 164.1668 105.6386) (end 164.1922 105.6132) (width 0.35) (layer F.Cu) (net 13) (status 30))
   (segment (start 164.1028 103.2256) (end 165.0238 103.2256) (width 0.35) (layer F.Cu) (net 13) (status 30))
-  (segment (start 144.5514 123.4694) (end 139.7 123.4694) (width 0.35) (layer B.Cu) (net 14))
-  (segment (start 135.7884 98.1202) (end 133.985 99.9236) (width 0.35) (layer F.Cu) (net 14))
+  (segment (start 144.5514 123.4694) (end 139.7 123.4694) (width 1) (layer B.Cu) (net 14))
+  (segment (start 135.7884 98.1202) (end 133.985 99.9236) (width 1) (layer F.Cu) (net 14))
   (via (at 135.7884 98.1202) (size 0.6) (drill 0.4) (layers F.Cu B.Cu) (net 14))
-  (segment (start 137.8204 100.1522) (end 135.7884 98.1202) (width 0.35) (layer B.Cu) (net 14))
-  (segment (start 137.8204 121.5898) (end 137.8204 100.1522) (width 0.35) (layer B.Cu) (net 14))
-  (segment (start 139.7 123.4694) (end 137.8204 121.5898) (width 0.35) (layer B.Cu) (net 14))
+  (segment (start 137.8204 100.1522) (end 135.7884 98.1202) (width 1) (layer B.Cu) (net 14))
+  (segment (start 137.8204 121.5898) (end 137.8204 100.1522) (width 1) (layer B.Cu) (net 14))
+  (segment (start 139.7 123.4694) (end 137.8204 121.5898) (width 1) (layer B.Cu) (net 14))
   (segment (start 133.985 99.9236) (end 133.985 101.502) (width 0.35) (layer F.Cu) (net 14))
   (segment (start 163.3474 115.951) (end 170.8404 115.951) (width 1) (layer B.Cu) (net 14))
-  (segment (start 172.3578 113.2144) (end 170.4594 113.2144) (width 0.5) (layer F.Cu) (net 14))
+  (segment (start 172.3578 113.2144) (end 170.4594 113.2144) (width 1) (layer F.Cu) (net 14))
   (segment (start 172.3898 113.1824) (end 172.3578 113.2144) (width 0.5) (layer F.Cu) (net 14))
   (via (at 172.3898 113.1824) (size 0.6) (drill 0.4) (layers F.Cu B.Cu) (net 14))
@@
   (segment (start 154.0866 104.5566) (end 154.1272 104.5972) (width 0.35) (layer F.Cu) (net 21))
   (segment (start 153.9654 103.4644) (end 153.7614 103.4644) (width 0.35) (layer F.Cu) (net 21) (status 30))
-  (zone (net 1) (net_name GND) (layer F.Cu) (hatch edge 0.508)
-    (connect_pads (clearance 0.508))
+  (zone (net 1) (net_name GND) (layer B.Cu) (hatch edge 0.508)
+    (connect_pads (clearance 0.8))
     (min_thickness 0.254)
     (fill yes (arc_segments 16) (thermal_gap 0.508) (thermal_bridge_width 0.508))
     (polygon
       (pts
-        (xy 131.3688 60.5536) (xy 176.9364 60.5536) (xy 176.9364 126.1364) (xy 131.3942 126.1364)
+        (xy 131.4196 60.6298) (xy 176.8856 60.5536) (xy 176.9364 126.111) (xy 131.3942 126.1364) (xy 131.4196 125.7808)
       )
     )
   )
-  (zone (net 1) (net_name GND) (layer B.Cu) (hatch edge 0.508)
-    (connect_pads (clearance 0.508))
+  (zone (net 1) (net_name GND) (layer F.Cu) (hatch edge 0.508)
+    (connect_pads (clearance 0.8))
     (min_thickness 0.254)
     (fill yes (arc_segments 16) (thermal_gap 0.508) (thermal_bridge_width 0.508))
     (polygon
       (pts
-        (xy 131.3688 60.5536) (xy 176.9364 60.5536) (xy 176.9364 126.1364) (xy 131.3942 126.1364)
+        (xy 131.4196 60.6298) (xy 176.8856 60.5536) (xy 176.9364 126.111) (xy 131.3942 126.1364) (xy 131.5974 125.857)
       )
     )
