File: BMS-Cell-Module-Circuit/BMS_Cell_Module.sch (KiCad schematic (older format))
At the start: 31 parts, among them J1 Conn_01x02_Female, J2 Conn_01x04_Female, J3 Conn_01x04_Female, M1 SI2312BDS-T1-E3, U2 ADUM1250ARZ, U3 ATTINY85V-10SU 8S2 EIAJ SOIC

Commit message: Minor amends
Parts:
- added TP2: TPGND, Connectors:PINTST, symbol TEST
Connections:
- wire segments 111 -> 112
Changed lines of the file:
@@
 Sheet 1 1
 Title "DIYBMS CELL MODULE"
-Date "2017-12-03"
+Date "2018-03-15"
 Rev "2"
 Comp ""
@@
 Text Notes 1760 3280 0    60   ~ 0
 For C1/C2/C6 Surface-mount ceramic types. \nIn all cases, X7R or X5R dielectric are recommended.
+$Comp
+L TEST TP2
+U 1 1 5A804029
+P 9990 5350
+F 0 "TP2" H 9990 5650 50  0000 C BNN
+F 1 "TPGND" H 9990 5600 50  0000 C CNN
+F 2 "Connectors:PINTST" H 9990 5350 50  0001 C CNN
+F 3 "" H 9990 5350 50  0001 C CNN
+	1    9990 5350
+	1    0    0    -1
+$EndComp
+Wire Wire Line
+	9990 5350 9990 5400
+Connection ~ 9990 5400
 $EndSCHEMATC

Commit message: Update R3 value in schematic to match pcb
In #5 I had set R3 to 68K based on the schematic value, rather than the 20k value on the PCB. This fixes the discrepancy.
Parts:
- R3: value 68K -> 20K
Changed lines of the file:
@@
 P 4200 5000
 F 0 "R3" V 4280 5000 50  0000 C CNN
-F 1 "68K" V 4100 5000 50  0000 C CNN
+F 1 "20K" V 4100 5000 50  0000 C CNN
 F 2 "Resistors_SMD:R_1206_HandSoldering" V 4130 5000 50  0001 C CNN
 F 3 "" H 4200 5000 50  0001 C CNN
